File: hardware/ILI2511-N7.kicad_pcb (KiCad board)
At the start: 2 copper layers, 40 x 25 mm, 31 parts, among them J1 FH35C-33S-0.3SHW, J2 FH35C-33S-0.3SHW, J3 I2C Touch, J4 USB_C_Receptacle_USB2.0, U1 ILITEK2511, U2 AP2112K-3.3, U3 USBLC6-2SC6, Y1 12MHz

Commit message: updated PCB footprint and new routing
Parts:
- removed REF**: OSHW-Logo2_9.8x8mm_SilkScreen, Symbol:OSHW-Logo2_9.8x8mm_SilkScreen
Other:
- board text added: "ddB0515 v3"
- board text removed: "ddB0515 v2"
